File: base/teensy_base_pcb/teensy_base_pcb.sch (KiCad schematic (older format))
At the start: 22 parts, among them Q1 PN2222A, U1 LM7805CT, U2 LD1117V33, U3 Teensy_3.2, U4 nRF24L01+

Commit message: PCB updates / clean up.
Parts:
- renumbered R3 to R1, R4 to R2
Connections:
- net NC: now also U3.21 (21/A7); no longer U3.3 (3(TX))
- net at P_SERVO1.1 (P1): now also U3.3 (3(TX)); no longer U3.21 (21/A7)
Changed lines of the file:
@@
 $EndComp
 $Comp
-L R R4
+L R R2
 U 1 1 58041CA0
 P 9650 3800
@@
 Text GLabel 5250 2150 0    60   UnSpc ~ 0
 NC
-Text GLabel 5250 2300 0    60   UnSpc ~ 0
+Text GLabel 7250 2450 2    60   UnSpc ~ 0
 NC
 Text GLabel 5250 2450 0    60   UnSpc ~ 0
@@
 $EndComp
 $Comp
-L R R3
+L R R1
 U 1 1 5803DA18
 P 2650 3900
@@
 	5500 4800 5450 4800
 Wire Wire Line
-	5450 4800 5450 4700
-Wire Wire Line
-	5450 4700 4750 4700
+	5450 4700 5450 4800
+Wire Wire Line
+	4750 4700 5450 4700
 Connection ~ 5250 4700
 Wire Wire Line
@@
 Wire Wire Line
 	3950 2100 3050 2100
-Wire Wire Line
-	7250 2450 8800 2450
-Wire Wire Line
-	8800 2450 8800 1650
 Wire Wire Line
 	8800 1650 10550 1650
@@
 Wire Wire Line
 	1500 2450 1600 2450
+Wire Wire Line
+	5250 2300 4900 2300
+Wire Wire Line
+	4900 2300 4900 900
+Wire Wire Line
+	4900 900  8800 900
+Wire Wire Line
+	8800 900  8800 1650
 $EndSCHEMATC

Commit message: Add accessory / future expansion ports to PCB.
Parts:
- added P_ACC1: CONN_01X03, Pin_Headers:Pin_Header_Straight_1x03, symbol CONN_01X03
- added P_ACC2: CONN_01X02, Pin_Headers:Pin_Header_Straight_1x02, symbol CONN_01X02
Connections:
- net +3.3V: now also P_ACC1.2 (P2)
- net +5V: now also P_ACC1.3 (P3)
- net GND: now also P_ACC1.1 (P1)
- net NC: no longer U3.16 (16/A2), U3.9 (9(RX2))
- new net ACC1: P_ACC2.2 (P2), U3.9 (9(RX2))
- new net ACC2: P_ACC2.1 (P1), U3.16 (16/A2)
Changed lines of the file:
@@
 Text GLabel 5250 2600 0    60   UnSpc ~ 0
 NC
-Text GLabel 5250 3200 0    60   UnSpc ~ 0
-NC
 Text GLabel 7250 1700 2    60   UnSpc ~ 0
 NC
@@
 NC
 Text GLabel 7250 3050 2    60   UnSpc ~ 0
-NC
-Text GLabel 7250 3200 2    60   UnSpc ~ 0
 NC
 Text GLabel 7250 3350 2    60   UnSpc ~ 0
@@
 	5500 4800 5450 4800
 Wire Wire Line
-	5450 4700 5450 4800
-Wire Wire Line
-	4750 4700 5450 4700
+	5450 4800 5450 4700
+Wire Wire Line
+	5450 4700 4750 4700
 Connection ~ 5250 4700
 Wire Wire Line
@@
 Wire Wire Line
 	8800 900  8800 1650
+$Comp
+L CONN_01X03 P_ACC1
+U 1 1 580AC98D
+P 850 3250
+F 0 "P_ACC1" H 850 3450 50  0000 R CNN
+F 1 "CONN_01X03" V 950 3250 50  0000 C CNN
+F 2 "Pin_Headers:Pin_Header_Straight_1x03" H 850 3250 50  0001 C CNN
+F 3 "" H 850 3250 50  0000 C CNN
+	1    850  3250
+	-1   0    0    1
+$EndComp
+$Comp
+L CONN_01X02 P_ACC2
+U 1 1 580ACB04
+P 850 3950
+F 0 "P_ACC2" H 850 4100 50  0000 R BNN
+F 1 "CONN_01X02" V 950 3950 50  0000 C CNN
+F 2 "Pin_Headers:Pin_Header_Straight_1x02" H 850 3950 50  0001 C CNN
+F 3 "" H 850 3950 50  0000 C CNN
+	1    850  3950
+	-1   0    0    1
+$EndComp
+Text GLabel 1300 3100 1    60   Input ~ 0
++5V
+Text GLabel 1300 3250 2    60   Input ~ 0
++3.3V
+$Comp
+L GND #PWR012
+U 1 1 580ACE3F
+P 1300 3450
+F 0 "#PWR012" H 1300 3200 50  0001 C CNN
+F 1 "GND" H 1300 3300 50  0000 C CNN
+F 2 "" H 1300 3450 50  0000 C CNN
+F 3 "" H 1300 3450 50  0000 C CNN
+	1    1300 3450
+	1    0    0    -1
+$EndComp
+Wire Wire Line
+	1050 3150 1300 3150
+Wire Wire Line
+	1300 3150 1300 3100
+Wire Wire Line
+	1050 3250 1300 3250
+Wire Wire Line
+	1050 3350 1300 3350
+Wire Wire Line
+	1300 3350 1300 3450
+Text GLabel 1300 3850 2    60   BiDi ~ 0
+ACC1
+Text GLabel 1300 4050 2    60   BiDi ~ 0
+ACC2
+Text GLabel 5250 3200 0    60   BiDi ~ 0
+ACC1
+Text GLabel 7250 3200 2    60   BiDi ~ 0
+ACC2
+Wire Wire Line
+	1300 4050 1050 4050
+Wire Wire Line
+	1050 4050 1050 4000
+Wire Wire Line
+	1300 3850 1050 3850
+Wire Wire Line
+	1050 3850 1050 3900
 $EndSCHEMATC

Commit message: Reverse PCB Acc 3.3 / 5V pins and clean up traces.
Connections:
- net +3.3V: now also P_ACC1.3 (P3); no longer P_ACC1.2 (P2)
- net +5V: now also P_ACC1.2 (P2); no longer P_ACC1.3 (P3)
Changed lines of the file:
@@
 	-1   0    0    1
 $EndComp
+Text GLabel 1300 3250 2    60   Input ~ 0
++5V
 Text GLabel 1300 3100 1    60   Input ~ 0
-+5V
-Text GLabel 1300 3250 2    60   Input ~ 0
 +3.3V
 $Comp

Commit message: Update schematic for motor driver / component.
Update capacitor footprints.
Parts:
- removed C1: 330nF, Capacitors_ThroughHole:C_Rect_L4_W2.5_P2.5, symbol C
- removed C4: 10uF, Capacitors_ThroughHole:C_Rect_L4_W2.5_P2.5, symbol C
- removed D1: 1N4004, Diodes_ThroughHole:Diode_DO-41_SOD81_Horizontal_RM10, symbol D
- removed Q1: PN2222A, TO_SOT_Packages_THT:TO-92_Inline_Narrow_Oval, symbol PN2222A
- removed R2: 270, Resistors_ThroughHole:Resistor_Horizontal_RM10mm, symbol R
- added C1: 330nF, Capacitors_ThroughHole:C_Rect_L7_W2.5_P5, symbol CP1
- added C4, C7: 10uF, Capacitors_ThroughHole:C_Radial_D5_L11_P2.5, symbol CP1
- added U5: TA8428K, Socket_Strips:Socket_Strip_Straight_1x07, symbol TA8428K
- C2, C3: footprint Capacitors_ThroughHole:C_Rect_L4_W2.5_P2.5 -> Capacitors_ThroughHole:C_Rect_L7_W2.5_P5
- C5: footprint Capacitors_ThroughHole:C_Radial_D10_L20_P5 -> Capacitors_ThroughHole:C_Radial_D8_L13_P3.8
- C6: footprint Capacitors_ThroughHole:C_Radial_D5_L11_P2 -> Capacitors_ThroughHole:C_Radial_D5_L11_P2.5
Connections:
- net +3.3V: now also C4.1
- net +9VA: now also C1.1, C7.1, U5.7 (VCC); no longer P_PUMP1.1 (P1)
- net GND: now also C1.2, C4.2, C7.2, U5.4 (GND)
- net NC: no longer U3.21 (21/A7)
- net at U3.20 (20/A6): now also U5.2 (IN2)
- net at P_PUMP1.2 (P2): now also U5.5 (-OUTA)
- new net: U3.21 (21/A7), U5.1 (IN1)
- new net: P_PUMP1.1 (P1), U5.3 (OUTA)
Changed lines of the file:
@@
 LIBS:nRF24L01+
 LIBS:ld1117v33
+LIBS:TA8428K
 LIBS:teensy_base_pcb-cache
 EELAYER 25 0
@@
 F 0 "C2" H 1675 6350 50  0000 L CNN
 F 1 "100nF" H 1675 6150 50  0000 L CNN
-F 2 "Capacitors_ThroughHole:C_Rect_L4_W2.5_P2.5" H 1688 6100 50  0001 C CNN
+F 2 "Capacitors_ThroughHole:C_Rect_L7_W2.5_P5" H 1688 6100 50  0001 C CNN
 F 3 "" H 1650 6250 50  0000 C CNN
 	1    1650 6250
-	1    0    0    -1
-$EndComp
-$Comp
-L C C1
-U 1 1 5803C1BB
-P 1650 5200
-F 0 "C1" H 1675 5300 50  0000 L CNN
-F 1 "330nF" H 1675 5100 50  0000 L CNN
-F 2 "Capacitors_ThroughHole:C_Rect_L4_W2.5_P2.5" H 1688 5050 50  0001 C CNN
-F 3 "" H 1650 5200 50  0000 C CNN
-	1    1650 5200
-	1    0    0    -1
-$EndComp
-$Comp
-L C C4
-U 1 1 5803C210
-P 3350 6250
-F 0 "C4" H 3375 6350 50  0000 L CNN
-F 1 "10uF" H 3375 6150 50  0000 L CNN
-F 2 "Capacitors_ThroughHole:C_Rect_L4_W2.5_P2.5" H 3388 6100 50  0001 C CNN
-F 3 "" H 3350 6250 50  0000 C CNN
-	1    3350 6250
 	1    0    0    -1
 $EndComp
@@
 F 0 "C3" H 3375 5300 50  0000 L CNN
 F 1 "100nF" H 3375 5100 50  0000 L CNN
-F 2 "Capacitors_ThroughHole:C_Rect_L4_W2.5_P2.5" H 3388 5050 50  0001 C CNN
+F 2 "Capacitors_ThroughHole:C_Rect_L7_W2.5_P5" H 3388 5050 50  0001 C CNN
 F 3 "" H 3350 5200 50  0000 C CNN
 	1    3350 5200
@@
 $EndComp
 $Comp
-L PN2222A Q1
-U 1 1 58041C1C
-P 10000 3800
-F 0 "Q1" H 10200 3875 50  0000 L CNN
-F 1 "PN2222A" H 10200 3800 50  0000 L CNN
-F 2 "TO_SOT_Packages_THT:TO-92_Inline_Narrow_Oval" H 10200 3725 50  0001 L CIN
-F 3 "" H 10000 3800 50  0000 L CNN
-	1    10000 3800
-	1    0    0    -1
-$EndComp
-$Comp
-L R R2
-U 1 1 58041CA0
-P 9650 3800
-F 0 "R2" V 9730 3800 50  0000 C CNN
-F 1 "270" V 9650 3800 50  0000 C CNN
-F 2 "Resistors_ThroughHole:Resistor_Horizontal_RM10mm" V 9580 3800 50  0001 C CNN
-F 3 "" H 9650 3800 50  0000 C CNN
-	1    9650 3800
-	0    1    1    0
-$EndComp
-$Comp
-L D D1
-U 1 1 58041DF8
-P 10300 3300
-F 0 "D1" H 10300 3400 50  0000 C CNN
-F 1 "1N4004" H 10300 3200 50  0000 C CNN
-F 2 "Diodes_ThroughHole:Diode_DO-41_SOD81_Horizontal_RM10" H 10300 3300 50  0001 C CNN
-F 3 "" H 10300 3300 50  0000 C CNN
-	1    10300 3300
-	-1   0    0    1
-$EndComp
-$Comp
 L CONN_01X03 P_SERVO1
 U 1 1 580427F1
@@
 F 0 "C5" H 10125 2000 50  0000 L CNN
 F 1 "470uF" H 10125 1800 50  0000 L CNN
-F 2 "Capacitors_ThroughHole:C_Radial_D10_L20_P5" H 10100 1900 50  0001 C CNN
+F 2 "Capacitors_ThroughHole:C_Radial_D8_L13_P3.8" H 10100 1900 50  0001 C CNN
 F 3 "" H 10100 1900 50  0000 C CNN
 	1    10100 1900
@@
 $EndComp
 Text GLabel 5250 2150 0    60   UnSpc ~ 0
-NC
-Text GLabel 7250 2450 2    60   UnSpc ~ 0
 NC
 Text GLabel 5250 2450 0    60   UnSpc ~ 0
@@
 L GND #PWR06
 U 1 1 5804FE02
-P 10100 4000
-F 0 "#PWR06" H 10100 3750 50  0001 C CNN
-F 1 "GND" H 10100 3850 50  0000 C CNN
-F 2 "" H 10100 4000 50  0000 C CNN
-F 3 "" H 10100 4000 50  0000 C CNN
-	1    10100 4000
-	1    0    0    -1
+P 8700 3600
+F 0 "#PWR06" H 8700 3350 50  0001 C CNN
+F 1 "GND" H 8700 3450 50  0000 C CNN
+F 2 "" H 8700 3600 50  0000 C CNN
+F 3 "" H 8700 3600 50  0000 C CNN
+	1    8700 3600
+	0    1    1    0
 $EndComp
 $Comp
@@
 Text GLabel 1600 2250 2    60   Output ~ 0
 +9V
-Text GLabel 10100 3050 0    60   Input ~ 0
+Text GLabel 8700 3900 0    60   Input ~ 0
 +9V
 Text GLabel 5000 5000 0    60   Input ~ 0
@@
 F 0 "C6" H 5275 4950 50  0000 L CNN
 F 1 "100uF" H 5275 4750 50  0000 L CNN
-F 2 "Capacitors_ThroughHole:C_Radial_D5_L11_P2" H 5250 4850 50  0001 C CNN
+F 2 "Capacitors_ThroughHole:C_Radial_D5_L11_P2.5" H 5250 4850 50  0001 C CNN
 F 3 "" H 5250 4850 50  0000 C CNN
 	1    5250 4850
@@
 Connection ~ 1650 6100
 Wire Wire Line
-	2800 6100 3550 6100
-Connection ~ 3350 6100
-Wire Wire Line
 	1050 6400 3350 6400
 Connection ~ 2500 6400
 Connection ~ 1650 6400
 Wire Wire Line
-	1050 5050 2100 5050
-Connection ~ 1650 5050
-Wire Wire Line
 	1050 5350 3350 5350
-Connection ~ 1650 5350
 Connection ~ 2500 5350
 Wire Wire Line
@@
 Connection ~ 3350 5050
 Wire Wire Line
-	10100 3600 10550 3600
-Wire Wire Line
 	7250 2600 8050 2600
-Wire Wire Line
-	8050 2600 8050 3800
-Wire Wire Line
-	8050 3800 9500 3800
 Wire Wire Line
 	10550 2050 10550 1850
@@
 Connection ~ 1500 2450
 Wire Wire Line
-	10150 3300 10100 3300
-Wire Wire Line
-	10100 3300 10100 3600
-Wire Wire Line
 	10550 5000 10100 5000
-Wire Wire Line
-	10550 3050 10100 3050
-Wire Wire Line
-	10550 3050 10550 3500
-Wire Wire Line
-	10450 3300 10550 3300
-Connection ~ 10550 3300
 Wire Wire Line
 	5500 5100 4600 5100
@@
 Wire Wire Line
 	1050 3850 1050 3900
+$Comp
+L TA8428K U5
+U 1 1 5813AE6C
+P 10050 3550
+F 0 "U5" H 10050 3300 60  0000 C CNN
+F 1 "TA8428K" H 10050 3800 60  0000 C CNN
+F 2 "Socket_Strips:Socket_Strip_Straight_1x07" H 10050 3550 60  0001 C CNN
+F 3 "" H 10050 3550 60  0001 C CNN
+	1    10050 3550
+	1    0    0    -1
+$EndComp
+Wire Wire Line
+	8050 2600 8050 3500
+Wire Wire Line
+	8050 3500 9550 3500
+Wire Wire Line
+	7250 2450 8150 2450
+Wire Wire Line
+	8150 2450 8150 3400
+Wire Wire Line
+	8150 3400 9550 3400
+Wire Wire Line
+	9350 3900 9350 3700
+Wire Wire Line
+	9350 3700 9550 3700
+$Comp
+L CP1 C7
+U 1 1 5813E1FE
+P 8900 3750
+F 0 "C7" H 8925 3850 50  0000 L CNN
+F 1 "10uF" H 8600 3750 50  0000 L CNN
+F 2 "Capacitors_ThroughHole:C_Radial_D5_L11_P2.5" H 8900 3750 50  0001 C CNN
+F 3 "" H 8900 3750 50  0000 C CNN
+	1    8900 3750
+	-1   0    0    1
+$EndComp
+Wire Wire Line
+	8700 3600 9550 3600
+Connection ~ 8900 3600
+Wire Wire Line
+	8700 3900 9350 3900
+Connection ~ 8900 3900
+$Comp
+L CP1 C4
+U 1 1 5813F531
+P 3350 6250
+F 0 "C4" H 3375 6350 50  0000 L CNN
+F 1 "10uF" H 3400 6150 50  0000 L CNN
+F 2 "Capacitors_ThroughHole:C_Radial_D5_L11_P2.5" H 3350 6250 50  0001 C CNN
+F 3 "" H 3350 6250 50  0000 C CNN
+	1    3350 6250
+	1    0    0    -1
+$EndComp
+Wire Wire Line
+	2800 6100 3550 6100
+Connection ~ 3350 6100
+$Comp
+L CP1 C1
+U 1 1 5813FD2B
+P 1650 5200
+F 0 "C1" H 1675 5300 50  0000 L CNN
+F 1 "330nF" H 1700 5100 50  0000 L CNN
+F 2 "Capacitors_ThroughHole:C_Rect_L7_W2.5_P5" H 1650 5200 50  0001 C CNN
+F 3 "" H 1650 5200 50  0000 C CNN
+	1    1650 5200
+	1    0    0    -1
+$EndComp
+Wire Wire Line
+	1050 5050 2100 5050
+Connection ~ 1650 5050
+Connection ~ 1650 5350
 $EndSCHEMATC

Commit message: Update PCB layout for TA8428K motor driver.
Parts:
- C4, C7: footprint Capacitors_ThroughHole:C_Radial_D5_L11_P2.5 -> Capacitors_ThroughHole:C_Rect_L7_W2.5_P5
- P_PUMP1: footprint Terminal_Blocks:TerminalBlock_Pheonix_MPT-2.54mm_2pol -> Terminal_Blocks:TerminalBlock_Pheonix_PT-3.5mm_2pol
Connections:
- net at U3.20 (20/A6): now also U5.1 (IN1); no longer U5.2 (IN2)
- net at U3.21 (21/A7): now also U5.2 (IN2); no longer U5.1 (IN1)
Changed lines of the file:
@@
 F 0 "P_PUMP1" H 10750 3700 50  0000 C BNN
 F 1 "CONN_01X02" V 10850 3550 50  0000 R CNN
-F 2 "Terminal_Blocks:TerminalBlock_Pheonix_MPT-2.54mm_2pol" H 10750 3550 50  0001 C CNN
+F 2 "Terminal_Blocks:TerminalBlock_Pheonix_PT-3.5mm_2pol" H 10750 3550 50  0001 C CNN
 F 3 "" H 10750 3550 50  0000 C CNN
 	1    10750 3550
@@
 $EndComp
 Wire Wire Line
-	8050 2600 8050 3500
-Wire Wire Line
-	8050 3500 9550 3500
-Wire Wire Line
 	7250 2450 8150 2450
-Wire Wire Line
-	8150 2450 8150 3400
-Wire Wire Line
-	8150 3400 9550 3400
 Wire Wire Line
 	9350 3900 9350 3700
@@
 F 0 "C7" H 8925 3850 50  0000 L CNN
 F 1 "10uF" H 8600 3750 50  0000 L CNN
-F 2 "Capacitors_ThroughHole:C_Radial_D5_L11_P2.5" H 8900 3750 50  0001 C CNN
+F 2 "Capacitors_ThroughHole:C_Rect_L7_W2.5_P5" H 8900 3750 50  0001 C CNN
 F 3 "" H 8900 3750 50  0000 C CNN
 	1    8900 3750
@@
 F 0 "C4" H 3375 6350 50  0000 L CNN
 F 1 "10uF" H 3400 6150 50  0000 L CNN
-F 2 "Capacitors_ThroughHole:C_Radial_D5_L11_P2.5" H 3350 6250 50  0001 C CNN
+F 2 "Capacitors_ThroughHole:C_Rect_L7_W2.5_P5" H 3350 6250 50  0001 C CNN
 F 3 "" H 3350 6250 50  0000 C CNN
 	1    3350 6250
@@
 Connection ~ 1650 5050
 Connection ~ 1650 5350
+Wire Wire Line
+	8150 2450 8150 3500
+Wire Wire Line
+	8150 3500 9550 3500
+Wire Wire Line
+	8050 2600 8050 3400
+Wire Wire Line
+	8050 3400 9550 3400
 $EndSCHEMATC

Commit message: Add resettable fuse / clean up traces / widths.
Parts:
- added F1: F_Small, Fuse_Holders_and_Fuses:Fuse_TE5_Littlefuse-395Series, symbol F_Small
Connections:
- net +9VA: now also F1.1; no longer C7.1, U5.7 (VCC)
- new net: C7.1, F1.2, U5.7 (VCC)
Changed lines of the file:
@@
 Text GLabel 1600 2250 2    60   Output ~ 0
 +9V
-Text GLabel 8700 3900 0    60   Input ~ 0
+Text GLabel 8400 3900 0    60   Input ~ 0
 +9V
 Text GLabel 5000 5000 0    60   Input ~ 0
@@
 Wire Wire Line
 	8050 3400 9550 3400
+$Comp
+L F_Small F1
+U 1 1 5814D4C0
+P 8600 3900
+F 0 "F1" H 8560 3960 50  0000 L CNN
+F 1 "F_Small" H 8480 3840 50  0000 L CNN
+F 2 "Fuse_Holders_and_Fuses:Fuse_TE5_Littlefuse-395Series" H 8600 3900 50  0001 C CNN
+F 3 "" H 8600 3900 50  0000 C CNN
+	1    8600 3900
+	1    0    0    -1
+$EndComp
+Wire Wire Line
+	8500 3900 8400 3900
 $EndSCHEMATC

Commit message: Swap servo output pins and clean up traces.
Connections:
- net GND: now also P_SERVO1.1 (P1); no longer P_SERVO1.3 (P3)
- net at U3.3 (3(TX)): now also P_SERVO1.3 (P3); no longer P_SERVO1.1 (P1)
Other:
- moved on the sheet: C5
Changed lines of the file:
@@
 L CP1 C5
 U 1 1 58042B68
-P 10100 1900
-F 0 "C5" H 10125 2000 50  0000 L CNN
-F 1 "470uF" H 10125 1800 50  0000 L CNN
-F 2 "Capacitors_ThroughHole:C_Radial_D8_L13_P3.8" H 10100 1900 50  0001 C CNN
-F 3 "" H 10100 1900 50  0000 C CNN
-	1    10100 1900
-	1    0    0    -1
+P 10100 1600
+F 0 "C5" H 10125 1700 50  0000 L CNN
+F 1 "470uF" H 10125 1500 50  0000 L CNN
+F 2 "Capacitors_ThroughHole:C_Radial_D8_L13_P3.8" H 10100 1600 50  0001 C CNN
+F 3 "" H 10100 1600 50  0000 C CNN
+	1    10100 1600
+	-1   0    0    1
 $EndComp
 Text GLabel 5250 2150 0    60   UnSpc ~ 0
@@
 L GND #PWR07
 U 1 1 58050A4E
-P 9600 2050
-F 0 "#PWR07" H 9600 1800 50  0001 C CNN
-F 1 "GND" H 9600 1900 50  0000 C CNN
-F 2 "" H 9600 2050 50  0000 C CNN
-F 3 "" H 9600 2050 50  0000 C CNN
-	1    9600 2050
+P 9600 1450
+F 0 "#PWR07" H 9600 1200 50  0001 C CNN
+F 1 "GND" H 9600 1300 50  0000 C CNN
+F 2 "" H 9600 1450 50  0000 C CNN
+F 3 "" H 9600 1450 50  0000 C CNN
+	1    9600 1450
 	1    0    0    -1
 $EndComp
@@
 	7250 2600 8050 2600
 Wire Wire Line
-	10550 2050 10550 1850
-Wire Wire Line
-	9600 2050 10550 2050
-Connection ~ 10100 2050
-Wire Wire Line
 	9600 1750 10550 1750
 Connection ~ 10100 1750
@@
 	5500 4800 5450 4800
 Wire Wire Line
-	5450 4800 5450 4700
-Wire Wire Line
-	5450 4700 4750 4700
+	5450 4700 5450 4800
+Wire Wire Line
+	4750 4700 5450 4700
 Connection ~ 5250 4700
 Wire Wire Line
@@
 Wire Wire Line
 	3950 2100 3050 2100
-Wire Wire Line
-	8800 1650 10550 1650
 Wire Wire Line
 	7250 2750 7650 2750
@@
 	4900 900  8800 900
 Wire Wire Line
-	8800 900  8800 1650
+	8800 900  8800 1850
 $Comp
 L CONN_01X03 P_ACC1
@@
 Wire Wire Line
 	8500 3900 8400 3900
+Wire Wire Line
+	10550 1450 10550 1650
+Wire Wire Line
+	9600 1450 10550 1450
+Connection ~ 10100 1450
+Wire Wire Line
+	8800 1850 10550 1850
 $EndSCHEMATC

Commit message: Move button resistor and more track clean up.
Connections:
- net +3.3V: now also P_ACC1.1 (P1); no longer P_ACC1.3 (P3)
- net GND: now also P_ACC1.3 (P3); no longer P_ACC1.1 (P1)
Changed lines of the file:
@@
 	5500 4800 5450 4800
 Wire Wire Line
-	5450 4700 5450 4800
-Wire Wire Line
-	4750 4700 5450 4700
+	5450 4800 5450 4700
+Wire Wire Line
+	5450 4700 4750 4700
 Connection ~ 5250 4700
 Wire Wire Line
@@
 Text GLabel 1300 3250 2    60   Input ~ 0
 +5V
-Text GLabel 1300 3100 1    60   Input ~ 0
+Text GLabel 1300 3450 2    60   Input ~ 0
 +3.3V
 $Comp
 L GND #PWR012
 U 1 1 580ACE3F
-P 1300 3450
-F 0 "#PWR012" H 1300 3200 50  0001 C CNN
-F 1 "GND" H 1300 3300 50  0000 C CNN
-F 2 "" H 1300 3450 50  0000 C CNN
-F 3 "" H 1300 3450 50  0000 C CNN
-	1    1300 3450
-	1    0    0    -1
-$EndComp
-Wire Wire Line
-	1050 3150 1300 3150
-Wire Wire Line
-	1300 3150 1300 3100
+P 1450 2950
+F 0 "#PWR012" H 1450 2700 50  0001 C CNN
+F 1 "GND" H 1450 2800 50  0000 C CNN
+F 2 "" H 1450 2950 50  0000 C CNN
+F 3 "" H 1450 2950 50  0000 C CNN
+	1    1450 2950
+	1    0    0    -1
+$EndComp
+Wire Wire Line
+	1300 3150 1050 3150
+Wire Wire Line
+	1300 2950 1300 3150
 Wire Wire Line
 	1050 3250 1300 3250
@@
 Wire Wire Line
 	8800 1850 10550 1850
+Wire Wire Line
+	1300 2950 1450 2950
 $EndSCHEMATC
